Commit message: Interface addition

File: urdf/motar_mini.urdf (robot description, URDF)
Before this commit: robot motar_mini, 17 links, 16 joints
Joints:
- joint wheel2: origin xyz=-0.07 -0.125 0.06 rpy=-2.9167 0 -1.5708 -> xyz=-0.07 -0.125 0.06 rpy=-2.2201 0 -1.5708

Commit message: tweaks

File: urdf/motar_mini.urdf (robot description, URDF)
Before this commit: robot motar_mini, 17 links, 16 joints
Links:
- link Wheel1: geometry collision cylinder length=0.05 radius=0.06; visual mesh filename=package://motar_mini/meshes/Wheel1.dae
- link Wheel2: geometry collision cylinder length=0.05 radius=0.06; visual mesh filename=package://motar_mini/meshes/Wheel2.dae
Joints:
- joint wheel1: origin xyz=-0.07 0.125 0.06 rpy=-2.2201 0 -1.5708 -> xyz=-0.07 0.155 0.06 rpy=-1.5708 0 -1.5708
- joint wheel2: origin xyz=-0.07 -0.125 0.06 rpy=-2.9167 0 -1.5708 -> xyz=-0.07 -0.125 0.06 rpy=-1.5708 0 -1.5708

Commit message: Reworked

File: urdf/motar_mini.urdf (robot description, URDF)
Before this commit: robot motar_mini, 17 links, 16 joints
Links:
- removed link Kapak
- removed link Mentese1
- removed link Mentese2
- removed link SWh1
- removed link SWh2
- removed link SWhSup1
- removed link SWhSup2
- removed link SWheel1
- removed link SWheel2
- removed link US1
- removed link US2
- removed link US3
- removed link Wheel1
- removed link Wheel2
- added link SF, mass 0.2; collision mesh filename=package://motar_mini/meshes/SF.STL; visual mesh filename=package://motar_mini/meshes/SF.STL
- added link SL, mass 0.2; collision mesh filename=package://motar_mini/meshes/SL.STL; visual mesh filename=package://motar_mini/meshes/SL.STL
- added link SR, mass 0.2; collision mesh filename=package://motar_mini/meshes/SR.STL; visual mesh filename=package://motar_mini/meshes/SR.STL
- added link SWhDir, mass 0.5; collision mesh filename=package://motar_mini/meshes/SWhDir.STL; visual mesh filename=package://motar_mini/meshes/SWhDir.STL
- added link SWheel, mass 1; collision mesh filename=package://motar_mini/meshes/SWheel.STL; visual mesh filename=package://motar_mini/meshes/SWheel.STL
- added link SWheelbase, mass 0.2; collision mesh filename=package://motar_mini/meshes/SWheelbase.STL; visual mesh filename=package://motar_mini/meshes/SWheelbase.STL
- added link leftWheel, mass 1; collision mesh filename=package://motar_mini/meshes/leftWheel.STL; visual mesh filename=package://motar_mini/meshes/leftWheel.STL
- added link rightWheel, mass 1; collision mesh filename=package://motar_mini/meshes/rightWheel.STL; visual mesh filename=package://motar_mini/meshes/rightWheel.STL
- link Dolap: mass 10 -> 5
- link base_link: mass 3.67445198488708 -> 3
- link hokuyo_link: geometry collision mesh filename=package://motar_mini/meshes/lidar.STL; visual mesh filename=package://motar_mini/meshes/lidar.STL
Joints:
- removed joint dolap
- removed joint kapak
- removed joint mentese1
- removed joint mentese2
- removed joint splate1
- removed joint splate2
- removed joint swheel1
- removed joint swheel2
- removed joint swhsup1
- removed joint swhsup2
- removed joint us1
- removed joint us2
- removed joint us3
- removed joint wheel1
- removed joint wheel2
- added joint Dolap: type fixed, parent base_link, child Dolap, origin xyz=0.152 -0.085 0.166002668970508 rpy=0 0 0, axis 0 0 0
- added joint LWheel: type continuous, parent base_link, child leftWheel, origin xyz=0.0858451267270673 0.0181457276792751 0.060002668970508 rpy=0 0 0, axis 0 1 0
- added joint RWheel: type continuous, parent base_link, child rightWheel, origin xyz=0.0858451267270673 -0.187145727679275 0.060002668970508 rpy=0 0 0, axis 0 1 0
- added joint SF: type fixed, parent base_link, child SF, origin xyz=0.299 -0.085 0.101002668970508 rpy=0 0 0, axis 0 0 0
- added joint SL: type fixed, parent base_link, child SL, origin xyz=0.276499221592938 -0.167500778407062 0.101002668970508 rpy=0 0 -0.785398163397448, axis 0 0 0
- added joint SR: type fixed, parent base_link, child SR, origin xyz=0.2765 -0.0025008 0.101 rpy=0 0 0.7854, axis 0 0 0
- added joint SWh: type continuous, parent SWhDir, child SWheel, origin xyz=-0.0177197511672673 -2.65387885129836E-05 -0.0136774048347897 rpy=0 0 0, axis 0.00149757402447565 -0.999998878635392 0
- added joint SWhBase: type fixed, parent base_link, child SWheelbase, origin xyz=0.272999999872566 -0.0849999999212055 0.039802668970508 rpy=0 0 0, axis 0 0 0
- added joint SWhD: type continuous, parent SWheelbase, child SWhDir, origin xyz=0.00221976872885976 0 -0.0104225951353673 rpy=0 0 0, axis 0 0 -1
- joint hokuyo_joint: origin xyz=0 0.00944754509525184 0.8256 rpy=0 0 0 -> xyz=0.145705213844625 -0.0898024549047488 0.618652668970508 rpy=0 0 0

Commit message: program updates

File: urdf/motar_mini.urdf (robot description, URDF)
Before this commit: robot motar_mini, 11 links, 10 joints
Links:
- link Dolap: mass 5 -> 10
- link SF: mass 0.2 -> 2
- link SL: mass 0.2 -> 2
- link SR: mass 0.2 -> 2
- link SWheel: mass 1 -> 0.5
- link SWheelbase: mass 0.2 -> 0.5
- link base_link: mass 3 -> 5
